File: pcb/zero_resistance_ammeter.sch (KiCad schematic (older format))
At the start: 18 parts

Commit message: associate footprints
Parts:
- removed BT?: Battery, TerminalBlock:TerminalBlock_bornier-2_P5.08mm, symbol Device:Battery
- removed Q?: TIP31A, Package_TO_SOT_THT:TO-220-3_Vertical, symbol Transistor_BJT:TIP41
- added BT1, BT2: Battery_Cell, Connector_PinHeader_2.54mm:PinHeader_1x02_P2.54mm_Vertical, symbol Device:Battery_Cell
- added C2: 100n, Capacitor_THT:C_Rect_L7.0mm_W2.5mm_P5.00mm, symbol Device:C
- added Q1: 2SD636, Connector_PinHeader_2.54mm:PinHeader_1x03_P2.54mm_Vertical, symbol Device:Q_NPN_ECB
- C1, C3, C4: renamed from C?; footprint (none) -> Capacitor_THT:C_Rect_L7.0mm_W2.5mm_P5.00mm
- D1: renamed from D?; value D_Schottky -> 1N5818; footprint (none) -> Diode_THT:D_DO-15_P10.16mm_Horizontal
- R1, R2, R3, R5, R6, R7: renamed from R?; footprint (none) -> Resistor_THT:R_Axial_DIN0207_L6.3mm_D2.5mm_P10.16mm_Horizontal
- R4: renamed from R?; value R -> 0.1R; footprint (none) -> PL_Resistor_SMD:R_2512
- RV1: renamed from RV?; footprint (none) -> Potentiometer_THT:Potentiometer_Bourns_3005_Horizontal
- gave numbers to parts that had none: 2
Connections:
- net GND: now also BT1.2 (-), BT2.1 (+), C2.1; no longer U1.4 (V-)
- net at C3.2, R2.1: now also Q1.3 (B)
- net at D1.2 (A): now also Q1.1 (E)
- net VCC renamed +BATT
- net +BATT: now also BT1.1 (+), Q1.2 (C)
- new net -BATT: BT2.2 (-), C2.2, U1.4 (V-)
Other:
- moved on the sheet: C1, U1C
